File: hardware/station_meteo.kicad_pcb (KiCad board)
At the start: 2 copper layers, 63.5 x 78.7 mm, 17 parts, among them J2 SSD1306 OLED, J3 DHT22, J4 DC Power, U1 ATmega328P-P, U2 LD1117S50TR_SOT223, Y1 16MHz

Commit message: Ajout
Parts:
- removed the C4 at (119.0, 45.7)
- removed U2: LD1117S50TR_SOT223, Package_TO_SOT_SMD:SOT-223-3_TabPin2
- added R3: 10k, Resistor_THT:R_Axial_DIN0204_L3.6mm_D1.6mm_P5.08mm_Horizontal, F.Cu at (116.8, 94.0)
- added U3: L7805, L385cv:TO255P1040X460X1968-3, F.Cu at (114.3, 33.0)
- C3: value 47 uf -> 100 nf; footprint Capacitor_SMD:CP_Elec_5x5.3 -> Capacitor_THT:C_Disc_D3.4mm_W2.1mm_P2.50mm
- C4: renamed from C5; value 0.1 uf -> 100 nf
- D2: footprint LED_SMD:LED_0805_2012Metric_Pad1.15x1.40mm_HandSolder -> LED_THT:LED_D3.0mm_Horizontal_O1.27mm_Z2.0mm
- U1: footprint Package_DIP:DIP-28_W7.62mm -> Package_DIP:DIP-28_W7.62mm_Socket
- moved C4 7.58 mm to (119.4, 45.7)
- moved C3 0.38 mm to (106.7, 45.7)
Connections:
- J2 pad 2: unconnected-(J2-Pin_2-Pad2) -> Net-(J2-Pin_2)
- J3 pad 2: Data -> Net-(J3-Pin_2)
- R5 pad 1: unconnected-(R5-Pad1) -> Net-(J2-Pin_2)
- R5 pad 2: unconnected-(R5-Pad2) -> SCL
Other:
- board size 63.5 x 78.7 mm -> 66 x 78.7 mm
