File: hardware/station_meteo.kicad_sch (KiCad schematic)
At the start: 17 parts, among them J2 SSD1306 OLED, J3 DHT22, J4 DC Power, U1 ATmega328P-P, U2 LD1117S50TR_SOT223, Y1 16MHz

Commit message: Ajout
Parts:
- removed C3, C4: 47 uf, Capacitor_SMD:CP_Elec_5x5.3, symbol Device:C_Polarized
- removed U2: LD1117S50TR_SOT223, Package_TO_SOT_SMD:SOT-223-3_TabPin2, symbol Regulator_Linear:LD1117S50TR_SOT223
- added C3: 100 nf, Capacitor_THT:C_Disc_D3.4mm_W2.1mm_P2.50mm, symbol Device:C
- added R3: 10k, Resistor_THT:R_Axial_DIN0204_L3.6mm_D1.6mm_P5.08mm_Horizontal, symbol Device:R
- added U3: L7805, L385cv:TO255P1040X460X1968-3, symbol Regulator_Linear:L7805
- C4: renamed from C5; value 0.1 uf -> 100 nf
- D2: footprint LED_SMD:LED_0805_2012Metric_Pad1.15x1.40mm_HandSolder -> LED_THT:LED_D3.0mm_Horizontal_O1.27mm_Z2.0mm
- U1: footprint Package_DIP:DIP-28_W7.62mm -> Package_DIP:DIP-28_W7.62mm_Socket
Connections:
- net +5V: now also U3.3 (OUT)
- net Data: now also R3.2; no longer J3.2 (Pin_2)
- net GND: now also C3.2, U3.2 (GND)
- net SCL: now also R5.2
- net at D1.1 (K): now also C3.1, U3.1 (IN)
- net at J2.2 (Pin_2): now also R5.1
- new net: J3.2 (Pin_2), R3.1
Other:
- moved on the sheet: C4
